File: hardware/hl/hermeslite.kicad_pcb (KiCad board)
At the start: 4 copper layers, 99.9 x 100 mm, 490 parts, among them CN1 USBBlaster2, CN10 RFD2b, CN2 PS, CN3 MagJack, CN4 STEREO, CN7 PS, CN8 RFD2b, CN9 RFD2b, J1 JNC, J10 JNC, J11 JNC, J12 JNO, J13 JNC, J14 JNC, J15 JNC, J16 JNO, J17 JNC, J18 JNC, J19 JNC, J2 JNC, J20 JNO, J21 JNC, J22 JNC, J23 JNC, J24 JNC, J25 JNC, J26 JNC, J27 JNC, J28 JNC, J29 JNC, J3 JNO, J30 JNC, J31 JNC, J32 JNC, J4 JNO, J5 JNC, J6 RFD2b, J7 JNO, J8 JNO, J9 JNC, K2 NA3WK-K, Q1 DMP3099L, Q2 NUD3124, Q3 LDMOS, Q4 LDMOS, Q5 NUD3124, Q6 MCP9700, T1 1:1 Z, T2 8:1 Z, T3 4:1 Z, U1 EEPROM, U10 PE4259, U11 PE4259, U12 AP2204, U13 MAX11613, U14 INA199A1DC, U15 MCP4662, U16 ST1S10, U17 TPS730, U19 LP2985, U2 FPGA, U3 ST1S10, U4 KSZ9031RN, U6 5P49V5923, U7 AD9866BCPZ, U8 ST1S10, U9 OPA2677, X1 25MHz, X2 38.4MHz, X3 38.4MHz

Commit message: add: ibom
Other:
- net class Default removed
