File: hardware/companions/n2adr/n2adr.kicad_pcb (KiCad board)
At the start: 4 copper layers, 100 x 49.9 mm, 166 parts, among them CN1 Audio-Jack-2, CN2 Conn_01x20, CN3 SMA, CN4 SMA, CN5 CONN_01X03, J3 Conn_01x01, K1 EC2-3NU, K2 EC2-3NU, K3 EC2-3NU, K4 EC2-3NU, K5 EC2-3NU, K6 EC2-3NU, K7 EC2-3NU, P1 TST, P13 TST, P14 TST, P15 TST, P16 TST, P2 TST, P3 TST, P4 TST, P5 TST, P6 TST, P7 TST, P8 TST, U1 MCP23008, U2 ULN2003LV, U3 AD8692, U5 74LVC1G00

Commit message: add: ibom pream
Other:
- net class Default removed
